Commit message: 260424_1531 change: block color re-indexing for ood obj

File: data/blocks/block_pink_big_10.urdf (robot description, URDF)
Before this commit: robot block_blue, 1 links, 0 joints
Links:
- link base_link: geometry collision box size=0.1 0.05 0.05; visual box size=0.1 0.05 0.05

File: data/blocks/block_red_middle_8.urdf (robot description, URDF)
Before this commit: robot block_blue, 1 links, 0 joints
Links:
- link base_link: geometry collision box size=0.07 0.05 0.05; visual box size=0.07 0.05 0.05
